File: BoxLight.sch (KiCad schematic (older format))
At the start: 7 parts, among them SW1 BUTTON, U1 MAX16054, U2 LTC6995-1

Commit message: Finished layout. Ready to order.
Parts:
- added SW2: BATTERY, Diodes_SMD:D_SMB_Standard, symbol TEST_2P
- D1, SW1: footprint Resistors_THT:R_Axial_DIN0204_L3.6mm_D1.6mm_P2.54mm_Vertical -> Diodes_SMD:D_SMB_Standard
Connections:
- net +3V3: now also SW2.1
- net GND: now also SW2.2
- net Circuit_PWR: now reaches D1.1, U1.5 (OUT)
- net Circuit_PWR: now also R1.1, U2.5 (V+)
Other:
- moved on the sheet: SW1, U1
Changed lines of the file:
@@
 L MAX16054 U1
 U 1 1 5A8CA123
-P 3200 2800
-F 0 "U1" H 3250 2850 60  0000 C CNN
-F 1 "MAX16054" H 3450 2350 60  0000 C CNN
-F 2 "TO_SOT_Packages_SMD:SOT-23-6_Handsoldering" H 3200 2800 60  0001 C CNN
-F 3 "" H 3200 2800 60  0001 C CNN
-	1    3200 2800
+P 2600 2800
+F 0 "U1" H 2650 2850 60  0000 C CNN
+F 1 "MAX16054" H 2850 2350 60  0000 C CNN
+F 2 "TO_SOT_Packages_SMD:SOT-23-6_Handsoldering" H 2600 2800 60  0001 C CNN
+F 3 "" H 2600 2800 60  0001 C CNN
+	1    2600 2800
 	1    0    0    -1
 $EndComp
@@
 L TEST_2P SW1
 U 1 1 5A8CACCA
-P 2600 3050
-F 0 "SW1" H 2600 3110 50  0000 C CNN
-F 1 "BUTTON" H 2600 2980 50  0000 C CNN
-F 2 "Resistors_THT:R_Axial_DIN0204_L3.6mm_D1.6mm_P2.54mm_Vertical" H 2600 3050 50  0001 C CNN
-F 3 "" H 2600 3050 50  0001 C CNN
-	1    2600 3050
+P 2000 3050
+F 0 "SW1" H 2000 3110 50  0000 C CNN
+F 1 "BUTTON" H 2000 2980 50  0000 C CNN
+F 2 "Diodes_SMD:D_SMB_Standard" H 2000 3050 50  0001 C CNN
+F 3 "" H 2000 3050 50  0001 C CNN
+	1    2000 3050
 	1    0    0    -1
 $EndComp
@@
 L GND #PWR01
 U 1 1 5A8CAE0F
-P 3650 4150
-F 0 "#PWR01" H 3650 3900 50  0001 C CNN
-F 1 "GND" H 3650 4000 50  0000 C CNN
-F 2 "" H 3650 4150 50  0001 C CNN
-F 3 "" H 3650 4150 50  0001 C CNN
-	1    3650 4150
-	1    0    0    -1
-$EndComp
-Wire Wire Line
-	3000 3050 2800 3050
-Wire Wire Line
-	2400 3050 2400 4100
-Wire Wire Line
-	2400 4100 3650 4100
-Wire Wire Line
-	3650 3850 3650 4150
-Connection ~ 3650 4100
+P 3050 4150
+F 0 "#PWR01" H 3050 3900 50  0001 C CNN
+F 1 "GND" H 3050 4000 50  0000 C CNN
+F 2 "" H 3050 4150 50  0001 C CNN
+F 3 "" H 3050 4150 50  0001 C CNN
+	1    3050 4150
+	1    0    0    -1
+$EndComp
+Wire Wire Line
+	2400 3050 2200 3050
+Wire Wire Line
+	1800 3050 1800 4100
+Wire Wire Line
+	1800 4100 3050 4100
+Wire Wire Line
+	3050 3850 3050 4150
+Connection ~ 3050 4100
 $Comp
 L GND #PWR02
@@
 L +3V3 #PWR03
 U 1 1 5A8CAFB1
-P 3650 2350
-F 0 "#PWR03" H 3650 2200 50  0001 C CNN
-F 1 "+3V3" H 3650 2490 50  0000 C CNN
-F 2 "Wire_Pads:SolderWirePad_single_1-5mmDrill" H 3650 2350 50  0001 C CNN
-F 3 "" H 3650 2350 50  0001 C CNN
-	1    3650 2350
-	1    0    0    -1
-$EndComp
-Wire Wire Line
-	3650 2350 3650 2600
+P 3050 2350
+F 0 "#PWR03" H 3050 2200 50  0001 C CNN
+F 1 "+3V3" H 3050 2490 50  0000 C CNN
+F 2 "Wire_Pads:SolderWirePad_single_1-5mmDrill" H 3050 2350 50  0001 C CNN
+F 3 "" H 3050 2350 50  0001 C CNN
+	1    3050 2350
+	1    0    0    -1
+$EndComp
+Wire Wire Line
+	3050 2350 3050 2600
 $Comp
 L GND #PWR04
@@
 	1    0    0    -1
 $EndComp
-NoConn ~ 4200 3250
+NoConn ~ 3600 3250
 $Comp
 L GND #PWR05
@@
 	6350 2750 5000 2750
 Wire Wire Line
-	5000 2750 5000 3450
-Wire Wire Line
-	5000 3450 4200 3450
-Wire Wire Line
-	4350 3050 4200 3050
+	5000 3450 5000 2750
+Wire Wire Line
+	3600 3450 5000 3450
+Wire Wire Line
+	3600 3050 4350 3050
 $Comp
 L TEST_2P D1
@@
 F 0 "D1" H 4550 3110 50  0000 C CNN
 F 1 "RGB_LED" H 4550 2980 50  0000 C CNN
-F 2 "Resistors_THT:R_Axial_DIN0204_L3.6mm_D1.6mm_P2.54mm_Vertical" H 4550 3050 50  0001 C CNN
+F 2 "Diodes_SMD:D_SMB_Standard" H 4550 3050 50  0001 C CNN
 F 3 "" H 4550 3050 50  0001 C CNN
 	1    4550 3050
@@
 Text Notes 2650 1750 0    60   ~ 0
 Three components are off-board and connect with wires:\n*Battery holder\n*RGB LED\n*Momentary N.O. push button
+$Comp
+L TEST_2P SW2
+U 1 1 5A96C61F
+P 3400 2400
+F 0 "SW2" H 3400 2460 50  0000 C CNN
+F 1 "BATTERY" H 3400 2330 50  0000 C CNN
+F 2 "Diodes_SMD:D_SMB_Standard" H 3400 2400 50  0001 C CNN
+F 3 "" H 3400 2400 50  0001 C CNN
+	1    3400 2400
+	1    0    0    -1
+$EndComp
+Wire Wire Line
+	3200 2400 3050 2400
+Connection ~ 3050 2400
+Wire Wire Line
+	3600 2400 3600 2550
+$Comp
+L GND #PWR06
+U 1 1 5A96C6DF
+P 3600 2550
+F 0 "#PWR06" H 3600 2300 50  0001 C CNN
+F 1 "GND" H 3600 2400 50  0000 C CNN
+F 2 "" H 3600 2550 50  0001 C CNN
+F 3 "" H 3600 2550 50  0001 C CNN
+	1    3600 2550
+	1    0    0    -1
+$EndComp
+Text Label 6300 3250 0    60   ~ 0
+Circuit_PWR
+Text Label 3650 3050 0    60   ~ 0
+Circuit_PWR
 $EndSCHEMATC
